File: Rev.0/CAD/38c3PCBLEDC100R_Rev.0.kicad_pcb (KiCad board)
At the start: 2 copper layers, 100 x 100 mm, 23 parts, among them Q2 ZVNL110A, U1 WeMos_D1_mini

Commit message: some files added
Parts:
- removed the REF** at (150.0, 129.5)
- added +5V: +5V, TestPoint:TestPoint_THTPad_2.5x2.5mm_Drill1.2mm, F.Cu at (136.0, 77.7)
- added GND: GND, TestPoint:TestPoint_THTPad_2.5x2.5mm_Drill1.2mm, F.Cu at (136.0, 73.2)
- added REF**: SuE, Logo:SuE, F.Cu at (179.8, 94.9)
- added REF**: OSHW-Symbol_13.4x12mm_F.Mask, Logo:OSHW-Symbol_13.4x12mm_F.Mask, F.Cu at (150.0, 129.5)
- added REF**: 38c3_Logo, Logo:38c3_Logo, B.Cu at (176.2, 82.4)
- added REF**: Blob01, Blob:Blob01, B.Cu at (150.0, 122.9)
- moved Q2 0.40 mm to (128.1, 73.1)
- moved A1 0.05 mm to (151.3, 78.2)
Connections:
- A1 pad 2: Net-(U1-A0) -> Net-(U1-MOSI/D7)
- A1 pad 3: Net-(U1-D0) -> Net-(U1-MISO/D6)
- A1 pad 5: Net-(U1-MISO/D6) -> Net-(U1-D0)
- A1 pad 6: Net-(U1-MOSI/D7) -> Net-(U1-A0)
- A1 pad 7: Net-(A1-Vin) -> GND
- A1 pad 8: GND -> Net-(A1-GND)
- Q2 pad 2: Net-(A1-Vin) -> Net-(A1-GND)
- R2 pad 1: Net-(A1-Vin) -> Net-(A1-GND)
- U1 pad 8: Net-(A1-Vin) -> Net-(A1-GND)
Routing:
- net Net-(A1-Vin): track 75.0 -> 0.00 mm
- net Net-(A1-GND): track 0.00 -> 50.9 mm
- net Net-(Q2-S): track 57.0 -> 56.0 mm
Other:
- board text added: "2024 c3RE"
- board text added: "Mistrust authority - promote decentralization."
- board text removed: "2023 c3RE"
- board text removed: "Mistrust authority - promote decentralization"
