File: Rev.0/CAD/38c3PCBLEDC100R_Rev.0.kicad_sch (KiCad schematic)
At the start: 20 parts, among them Q2 ZVNL110A, U1 WeMos_D1_mini

Commit message: some files added
Parts:
- added H5: GND, TestPoint:TestPoint_THTPad_2.5x2.5mm_Drill1.2mm, symbol Mechanical:MountingHole_Pad
- added H6: +5V, TestPoint:TestPoint_THTPad_2.5x2.5mm_Drill1.2mm, symbol Mechanical:MountingHole_Pad
Connections:
- net +5V: now also H6.1
- net GND: now also A1.7 (GND), H5.1; no longer A1.8 (GND)
- net at Q2.2 (G), R2.1, U1.8 (3V3): now also A1.8 (Vin); no longer A1.7 (Vin)
- net at A1.2: now also U1.6 (MOSI/D7); no longer U1.2 (A0)
- net at A1.3: now also U1.5 (MISO/D6); no longer U1.3 (D0)
- net at A1.5: now also U1.3 (D0); no longer U1.5 (MISO/D6)
- net at A1.6: now also U1.2 (A0); no longer U1.6 (MOSI/D7)
Other:
- moved on the sheet: H3, H4
Changed lines of the file:
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@@
 	)
 	(junction
-		(at 177.8 107.95)
+		(at 177.8 128.27)
 		(diameter 0)
 		(color 0 0 0 0)
@@
 	)
 	(junction
-		(at 177.8 101.6)
+		(at 177.8 121.92)
 		(diameter 0)
 		(color 0 0 0 0)
@@
 	)
 	(junction
+		(at 177.8 115.57)
+		(diameter 0)
+		(color 0 0 0 0)
+	)
+	(junction
 		(at 182.88 55.88)
 		(diameter 0)
@@
 	)
 	(junction
+		(at 177.8 88.9)
+		(diameter 0)
+		(color 0 0 0 0)
+	)
+	(junction
 		(at 59.69 45.72)
 		(diameter 0)
@@
 	(wire
 		(pts
+			(xy 177.8 109.22) (xy 177.8 115.57)
+		)
+		(stroke
+			(width 0)
+			(type default)
+		)
+	)
+	(wire
+		(pts
 			(xy 146.05 99.06) (xy 148.59 99.06)
 		)
@@
 	(wire
 		(pts
-			(xy 170.18 107.95) (xy 177.8 107.95)
+			(xy 170.18 128.27) (xy 177.8 128.27)
 		)
 		(stroke
@@
 	(wire
 		(pts
+			(xy 180.34 109.22) (xy 177.8 109.22)
+		)
+		(stroke
+			(width 0)
+			(type default)
+		)
+	)
+	(wire
+		(pts
 			(xy 231.14 35.56) (xy 231.14 45.72)
 		)
@@
 	(wire
 		(pts
+			(xy 177.8 95.25) (xy 177.8 88.9)
+		)
+		(stroke
+			(width 0)
+			(type default)
+		)
+	)
+	(wire
+		(pts
 			(xy 109.22 104.14) (xy 109.22 93.98)
 		)
@@
 	(wire
 		(pts
+			(xy 180.34 95.25) (xy 177.8 95.25)
+		)
+		(stroke
+			(width 0)
+			(type default)
+		)
+	)
+	(wire
+		(pts
 			(xy 125.73 35.56) (xy 144.78 35.56)
 		)
@@
 	(wire
 		(pts
-			(xy 177.8 95.25) (xy 180.34 95.25)
+			(xy 177.8 115.57) (xy 180.34 115.57)
 		)
 		(stroke
@@
 	(wire
 		(pts
-			(xy 170.18 113.03) (xy 170.18 107.95)
+			(xy 170.18 133.35) (xy 170.18 128.27)
 		)
 		(stroke
@@
 	(wire
 		(pts
-			(xy 177.8 107.95) (xy 177.8 101.6)
+			(xy 177.8 128.27) (xy 177.8 121.92)
 		)
 		(stroke
@@
 	(wire
 		(pts
-			(xy 177.8 101.6) (xy 180.34 101.6)
+			(xy 177.8 121.92) (xy 180.34 121.92)
 		)
 		(stroke
@@
 	(wire
 		(pts
-			(xy 177.8 101.6) (xy 177.8 95.25)
+			(xy 177.8 121.92) (xy 177.8 115.57)
 		)
 		(stroke
@@
 	(wire
 		(pts
-			(xy 177.8 107.95) (xy 177.8 113.03)
+			(xy 177.8 128.27) (xy 177.8 133.35)
 		)
 		(stroke
@@
 	(symbol
 		(lib_id "Mechanical:MountingHole_Pad")
-		(at 182.88 95.25 270)
+		(at 182.88 115.57 270)
 		(unit 1)
 		(exclude_from_sim no)
@@
 		(dnp no)
 		(property "Reference" "H3"
-			(at 186.69 93.98 90)
+			(at 186.69 114.3 90)
 			(effects
 				(font
@@
 		)
 		(property "Value" "GND"
-			(at 186.69 96.52 90)
+			(at 186.69 116.84 90)
 			(effects
 				(font
@@
 		)
 		(property "Footprint" "MountingHole:MountingHole_3.2mm_M3_DIN965_Pad"
-			(at 182.88 95.25 0)
+			(at 182.88 115.57 0)
 			(effects
 				(font
@@
 		)
 		(property "Datasheet" "~"
-			(at 182.88 95.25 0)
+			(at 182.88 115.57 0)
 			(effects
 				(font
@@
 		)
 		(property "Description" "Mounting Hole with connection"
-			(at 182.88 95.25 0)
+			(at 182.88 115.57 0)
 			(effects
 				(font
@@
 	(symbol
 		(lib_id "Mechanical:MountingHole_Pad")
-		(at 182.88 101.6 270)
+		(at 182.88 121.92 270)
 		(unit 1)
 		(exclude_from_sim no)
@@
 		(fields_autoplaced yes)
 		(property "Reference" "H4"
-			(at 186.69 100.965 90)
+			(at 186.69 121.285 90)
 			(effects
 				(font
@@
 		)
 		(property "Value" "GND"
-			(at 186.69 103.505 90)
+			(at 186.69 123.825 90)
 			(effects
 				(font
@@
 		)
 		(property "Footprint" "MountingHole:MountingHole_3.2mm_M3_DIN965_Pad"
-			(at 182.88 101.6 0)
+			(at 182.88 121.92 0)
 			(effects
 				(font
@@
 		)
 		(property "Datasheet" "~"
-			(at 182.88 101.6 0)
+			(at 182.88 121.92 0)
 			(effects
 				(font
@@
 		)
 		(property "Description" "Mounting Hole with connection"
-			(at 182.88 101.6 0)
+			(at 182.88 121.92 0)
 			(effects
 				(font
@@
 	(symbol
 		(lib_id "power:GND")
-		(at 177.8 113.03 0)
+		(at 177.8 133.35 0)
 		(unit 1)
 		(exclude_from_sim no)
@@
 		(fields_autoplaced yes)
 		(property "Reference" "#PWR02"
-			(at 177.8 119.38 0)
+			(at 177.8 139.7 0)
 			(effects
 				(font
@@
 		)
 		(property "Value" "GND"
-			(at 177.8 118.11 0)
+			(at 177.8 138.43 0)
 			(effects
 				(font
@@
 		)
 		(property "Footprint" ""
-			(at 177.8 113.03 0)
+			(at 177.8 133.35 0)
 			(effects
 				(font
@@
 		)
 		(property "Datasheet" ""
-			(at 177.8 113.03 0)
+			(at 177.8 133.35 0)
 			(effects
 				(font
@@
 		)
 		(property "Description" "Power symbol creates a global label with name \"GND\" , ground"
-			(at 177.8 113.03 0)
+			(at 177.8 133.35 0)
 			(effects
 				(font
@@
 	)
 	(symbol
+		(lib_id "Mechanical:MountingHole_Pad")
+		(at 182.88 95.25 270)
+		(unit 1)
+		(exclude_from_sim yes)
+		(in_bom no)
+		(on_board yes)
+		(dnp no)
+		(fields_autoplaced yes)
+		(property "Reference" "H6"
+			(at 186.69 93.9799 90)
+			(effects
+				(font
+					(size 1.27 1.27)
+				)
+				(justify left)
+			)
+		)
+		(property "Value" "+5V"
+			(at 186.69 96.5199 90)
+			(effects
+				(font
+					(size 1.27 1.27)
+				)
+				(justify left)
+			)
+		)
+		(property "Footprint" "TestPoint:TestPoint_THTPad_2.5x2.5mm_Drill1.2mm"
+			(at 182.88 95.25 0)
+			(effects
+				(font
+					(size 1.27 1.27)
+				)
+				(hide yes)
+			)
+		)
+		(property "Datasheet" "~"
+			(at 182.88 95.25 0)
+			(effects
+				(font
+					(size 1.27 1.27)
+				)
+				(hide yes)
+			)
+		)
+		(property "Description" "Mounting Hole with connection"
+			(at 182.88 95.25 0)
+			(effects
+				(font
+					(size 1.27 1.27)
+				)
+				(hide yes)
+			)
+		)
+		(pin "1"
+		)
+		(instances
+			(project ""
+				(path "/4acc92b7-ae78-4f6f-8f1d-403b41b8ff51"
+					(reference "H6")
+					(unit 1)
+				)
+			)
+		)
+	)
+	(symbol
 		(lib_id "WS2812D-F5-1261:WS2812D-F5-1261")
 		(at 163.83 45.72 0)
@@
 	)
 	(symbol
+		(lib_id "Mechanical:MountingHole_Pad")
+		(at 182.88 109.22 270)
+		(unit 1)
+		(exclude_from_sim yes)
+		(in_bom no)
+		(on_board yes)
+		(dnp no)
+		(fields_autoplaced yes)
+		(property "Reference" "H5"
+			(at 186.69 107.9499 90)
+			(effects
+				(font
+					(size 1.27 1.27)
+				)
+				(justify left)
+			)
+		)
+		(property "Value" "GND"
+			(at 186.69 110.4899 90)
+			(effects
+				(font
+					(size 1.27 1.27)
+				)
+				(justify left)
+			)
+		)
+		(property "Footprint" "TestPoint:TestPoint_THTPad_2.5x2.5mm_Drill1.2mm"
+			(at 182.88 109.22 0)
+			(effects
+				(font
+					(size 1.27 1.27)
+				)
+				(hide yes)
+			)
+		)
+		(property "Datasheet" "~"
+			(at 182.88 109.22 0)
+			(effects
+				(font
+					(size 1.27 1.27)
+				)
+				(hide yes)
+			)
+		)
+		(property "Description" "Mounting Hole with connection"
+			(at 182.88 109.22 0)
+			(effects
+				(font
+					(size 1.27 1.27)
+				)
+				(hide yes)
+			)
+		)
+		(pin "1"
+		)
+		(instances
+			(project ""
+				(path "/4acc92b7-ae78-4f6f-8f1d-403b41b8ff51"
+					(reference "H5")
+					(unit 1)
+				)
+			)
+		)
+	)
+	(symbol
 		(lib_id "WS2812D-F5-1261:WS2812D-F5-1261")
 		(at 182.88 45.72 0)
@@
 	(symbol
 		(lib_id "power:PWR_FLAG")
-		(at 170.18 113.03 180)
+		(at 170.18 133.35 180)
 		(unit 1)
 		(exclude_from_sim no)
@@
 		(fields_autoplaced yes)
 		(property "Reference" "#FLG02"
-			(at 170.18 114.935 0)
+			(at 170.18 135.255 0)
 			(effects
 				(font
@@
 		)
 		(property "Value" "PWR_FLAG"
-			(at 170.18 118.11 0)
+			(at 170.18 138.43 0)
 			(effects
 				(font
@@
 		)
 		(property "Footprint" ""
-			(at 170.18 113.03 0)
+			(at 170.18 133.35 0)
 			(effects
 				(font
@@
 		)
 		(property "Datasheet" "~"
-			(at 170.18 113.03 0)
+			(at 170.18 133.35 0)
 			(effects
 				(font
@@
 		)
 		(property "Description" "Special symbol for telling ERC where power comes from"
-			(at 170.18 113.03 0)
+			(at 170.18 133.35 0)
 			(effects
 				(font
